File: MegaDAQ_buffer-top.sch (KiCad schematic (older format))
At the start: 0 parts

Commit message: commiting version v1c, produced
Connections:
- net labels added: Ain_os0, Ain_os1, Ain_os10, Ain_os11, Ain_os12, Ain_os13, Ain_os14, Ain_os15, Ain_os2, Ain_os3, Ain_os4, Ain_os5, Ain_os6, Ain_os7, Ain_os8, Ain_os9, Ain_os[0..15]
- wire segments 92 -> 108
