File: MegaDAQ_buffering.sch (KiCad schematic (older format))
At the start: 20 parts, among them IC301 MC33079D

Commit message: commiting version v1c, produced
Parts:
- removed IC301: MC33079D, linear2-SO14, symbol MC33079D
- removed R301, R302, R303, R304, R305, R306, R307, R308: 10k, Resistors_SMD:R_0603, symbol R
- removed RP301: R_PACK8, Resistors_SMD:R_Cat16-8, symbol R_PACK8
- added C2, C3: 0.1u, Capacitors_SMD:C_0603, symbol C
- added R3, R4, R5, R6: 10k, Resistors_SMD:R_0603_HandSoldering, symbol R
- added U602, U603: diffamp, Housings_SOIC:SOIC-14_3.9x8.7mm_Pitch1.27mm, symbol diffamp
- C601: renamed from C301; value C -> 2n
- C602: renamed from C302; value C -> 2n
- C603: renamed from C303; value C -> 2n
- C604: renamed from C304; value C -> 2n
- R601: renamed from R309; value 10k -> 100; footprint Resistors_SMD:R_0603_HandSoldering -> Resistors_SMD:R_0603
- R602: renamed from R310; value 10k -> 100; footprint Resistors_SMD:R_0603_HandSoldering -> Resistors_SMD:R_0603
- R603: renamed from R311; value 10k -> 100; footprint Resistors_SMD:R_0603_HandSoldering -> Resistors_SMD:R_0603
- R604: renamed from R312; value 10k -> 100; footprint Resistors_SMD:R_0603_HandSoldering -> Resistors_SMD:R_0603
- renumbered C305 to C605, C306 to C606
Connections:
- net AIN+0: now also R3.2, U602.3 (+InA)
- net AIN+1: now also R4.2, U602.5 (+InB)
- net AIN+2: now also R5.2, U603.3 (+InA)
- net AIN+3: now also R6.2, U603.5 (+InB)
- net AIN-0: now also R3.1, U602.2 (-InA)
- net AIN-1: now also R4.1, U602.6 (-InB)
- net AIN-2: now also R5.1, U603.2 (-InA)
- net AIN-3: now also R6.1, U603.6 (-InB)
- net AV_CC: now also C2.1, U602.11 (V+), U603.11 (V+)
- net AV_EE: now also C3.2, U602.4 (V-), U603.4 (V-)
- net GNDA: now also C2.2, C3.1
- net at C601.1, R604.1: now also U602.12 (SensA), U602.13 (OutA)
- net at C602.1, R601.1: now also U602.10 (SensB), U602.9 (OutB)
- net at C603.1, R602.1: now also U603.12 (SensA), U603.13 (OutA)
- net at C604.1, R603.1: now also U603.10 (SensB), U603.9 (OutB)
- new net ADC_OFFSET_0: U602.14 (RefA)
- new net ADC_OFFSET_1: U602.8 (RefB)
- new net ADC_OFFSET_2: U603.14 (RefA)
- new net ADC_OFFSET_3: U603.8 (RefB)
