File: MegaDAQ_buffering_single-ended.sch (KiCad schematic (older format))
At the start: 16 parts, among them IC501 MC33079D

Commit message: commiting version v1c, produced
Parts:
- removed R505, R506, R507, R508: 10k, Resistors_SMD:R_0603, symbol R
- C301: renamed from C501; value C -> 10n
- C304: renamed from C502; value C -> 10n
- C305: renamed from C503; value C -> 10n
- C306: renamed from C504; value C -> 10n
- IC301: renamed from IC501; footprint linear2-SO14 -> Housings_SOIC:SOIC-14_3.9x8.7mm_Pitch1.27mm; manf# (none) -> MC33079DT
- R301: renamed from R501; value 10k -> 100
- R302: renamed from R502; value 10k -> 100
- R303: renamed from R503; value 10k -> 100
- R304: renamed from R504; value 10k -> 100
- RP301: renamed from RP501; value R_PACK4 -> R_PACK4 50R; manf# (none) -> CAT16-49R9F4LF
- renumbered C505 to C302, C506 to C303, IC501 to IC301
Connections:
- net OUT0: now also C301.1
- net OUT1: now also C304.1
- net OUT2: now also C305.1
- net OUT3: now also C306.1
- net at IC301.2 (-IN): now also IC301.1 (OUT), RP301.1 (P1)
- net at IC301.7 (OUT), RP301.2 (P2): now also IC301.6 (-IN); no longer C304.1
- net at IC301.8 (OUT), RP301.3 (P3): now also IC301.9 (-IN); no longer C305.1
- net at IC301.14 (OUT), RP301.4 (P4): now also IC301.13 (-IN); no longer C306.1
Other:
- moved on the sheet: C301, C304, C305, C306
