File: megaDAQ.kicad_pcb (KiCad board)
At the start: 2 copper layers, 123.2 x 100 mm, 148 parts, among them IC301 MC33079D, IC401 MC33079D, IC501 MC33079D, IC601 MC33079D, IC701 MC33079D, IC801 MC33079D, IC901 MC33079D, P101 CONN_02X03, P102 CONN_02X30, P103 CONN_01X01, P104 CONN_01X01, P105 CONN_01X01, P106 CONN_02X18, P107 CONN_01X10, P108 CONN_01X08, P109 CONN_01X08, P112 CONN_01X01, P114 CONN_01X01, U101 AMC7812SPAPR, U102 LM78M05CT

Commit message: commiting version v1c, produced
Parts:
- removed IC601, IC701, IC801, IC901: MC33079D, Housings_SOIC:SOIC-14_3.9x8.7mm_Pitch1.27mm
- removed P101: CONN_02X03, Pin_Headers:Pin_Header_Straight_2x03
- removed P103, P104: CONN_01X01, screw_terminals:keystone_7773
- removed P107: CONN_01X10, Pin_Headers:Pin_Header_Straight_1x10
- removed P108, P109: CONN_01X08, Pin_Headers:Pin_Header_Straight_1x08
- removed P112, P114: CONN_01X01, Connect:1pin
- removed R305, R306, R307, R308, R405, R406, R407, R408, R505, R506, R507, R508, R605, R606, R607, R608, R705, R706, R707, R708, R805, R806, R807, R808, R905, R906, R907, R908: 10k, Resistors_SMD:R_0603
- removed R309, R310, R311, R312, R409, R410, R411, R412, R609, R610, R611, R612, R709, R710, R711, R712: 10k, Resistors_SMD:R_0603_HandSoldering
- removed RP601, RP701: R_PACK8, Resistors_SMD:R_Cat16-8
- removed RP801, RP901: R_PACK4, Resistors_SMD:R_Cat16-4
- added C1: 15u, SMD_Packages:SMD-1206_Pol, F.Cu at (124.4, 80.9)
- added C1001: 100n, Capacitors_SMD:C_0603, F.Cu at (127.3, 77.7)
- added C1002: 100n, Capacitors_SMD:C_0603, F.Cu at (139.4, 77.1)
- added C1003: 1n, Capacitors_SMD:C_0603, F.Cu at (127.5, 73.2)
- added C1004: 100n, Capacitors_SMD:C_0603, F.Cu at (128.4, 63.5)
- added C1101: 100n, Capacitors_SMD:C_0603, F.Cu at (108.9, 64.9)
- added C1102: 100n, Capacitors_SMD:C_0603, F.Cu at (99.1, 64.9)
- added C2: 0.1u, Capacitors_SMD:C_0603, F.Cu at (77.2, 112.0)
- added C3: 0.1u, Capacitors_SMD:C_0603, F.Cu at (64.5, 112.0)
- added C4: 0.1u, Capacitors_SMD:C_0603, F.Cu at (58.0, 99.5)
- added C5: 0.1u, Capacitors_SMD:C_0603, F.Cu at (45.5, 87.0)
- added C6: 0.1u, Capacitors_SMD:C_0603, F.Cu at (58.0, 87.0)
- added C7: 0.1u, Capacitors_SMD:C_0603, F.Cu at (45.5, 99.5)
- added C8: 0.1u, Capacitors_SMD:C_0603, F.Cu at (58.0, 74.5)
- added C9: 0.1u, Capacitors_SMD:C_0603, F.Cu at (45.5, 74.5)
- added D1: BAS16, Diodes_SMD:SOD-523, F.Cu at (124.2, 73.2)
- added D1001: BAS16, Diodes_SMD:SOD-523, F.Cu at (127.9, 66.5)
- added IC1001: MC33079D, Housings_SOIC:SOIC-14_3.9x8.7mm_Pitch1.27mm, F.Cu at (133.4, 77.1)
- added Q1001: PZT2222A, TO_SOT_Packages_SMD:SOT-223, F.Cu at (136.0, 67.1)
- added R1: 698, Resistors_SMD:R_0603, F.Cu at (121.0, 75.3)
- added R10: DNI, Resistors_SMD:R_0603_HandSoldering, F.Cu at (64.2, 89.2)
- added R1001: 100, Resistors_SMD:R_0603, F.Cu at (127.5, 75.3)
- added R1002: 100, Resistors_SMD:R_0603, F.Cu at (129.1, 69.2)
- added R1003: 500, Resistors_SMD:R_0603, F.Cu at (126.7, 69.2)
- added R1004: 10k, Resistors_SMD:R_0603, F.Cu at (138.7, 72.6)
- added R11: DNI, Resistors_SMD:R_0603_HandSoldering, F.Cu at (45.0, 97.5)
- added R1101: 0, Resistors_SMD:R_0603_HandSoldering, B.Cu at (117.3, 83.7)
- added R1102: DNI, Resistors_SMD:R_0603_HandSoldering, B.Cu at (114.3, 83.7)
- added R1103: DNI, Resistors_SMD:R_0603_HandSoldering, B.Cu at (122.3, 89.0)
- added R1104: 0, Resistors_SMD:R_0603_HandSoldering, B.Cu at (119.3, 89.0)
- added R1105: DNI, Resistors_SMD:R_0603_HandSoldering, B.Cu at (119.5, 99.5)
- added R1106: 0, Resistors_SMD:R_0603_HandSoldering, B.Cu at (116.5, 99.5)
- added R1107: 0, Resistors_SMD:R_0603_HandSoldering, B.Cu at (108.8, 83.7)
- added R1108: DNI, Resistors_SMD:R_0603_HandSoldering, B.Cu at (105.8, 83.7)
- added R1109: DNI, Resistors_SMD:R_0603_HandSoldering, B.Cu at (108.8, 89.7)
- added R1110: 0, Resistors_SMD:R_0603_HandSoldering, B.Cu at (105.7, 89.7)
- added R1111: 0, Resistors_SMD:R_0603_HandSoldering, B.Cu at (108.8, 95.8)
- added R1112: DNI, Resistors_SMD:R_0603_HandSoldering, B.Cu at (105.7, 95.8)
- added R1113: 10k, Resistors_SMD:R_0603, F.Cu at (56.5, 67.6)
- added R1114: 10k, Resistors_SMD:R_0603, F.Cu at (56.5, 64.7)
- added R1115: 10k, Resistors_SMD:R_0603, F.Cu at (71.6, 67.6)
- added R1116: 10k, Resistors_SMD:R_0603, F.Cu at (71.6, 64.7)
- added R1117: 10k, Resistors_SMD:R_0603, F.Cu at (76.5, 67.6)
- added R1118: 10k, Resistors_SMD:R_0603, F.Cu at (76.5, 64.7)
- added R1119: 10k, Resistors_SMD:R_0603, F.Cu at (61.6, 64.7)
- added R1120: 10k, Resistors_SMD:R_0603, F.Cu at (61.6, 67.6)
- added R1121: 10k, Resistors_SMD:R_0603, F.Cu at (66.4, 64.7)
- added R1122: 10k, Resistors_SMD:R_0603, F.Cu at (66.4, 67.6)
- added R1123: 10k, Resistors_SMD:R_0603, F.Cu at (81.8, 64.7)
- added R1124: 10k, Resistors_SMD:R_0603, F.Cu at (81.8, 67.6)
- added R1125: 10k, Resistors_SMD:R_0603, F.Cu at (86.5, 67.6)
- added R1126: 10k, Resistors_SMD:R_0603, F.Cu at (86.5, 64.8)
- added R1127: 10k, Resistors_SMD:R_0603, F.Cu at (51.4, 64.7)
- added R1128: 10k, Resistors_SMD:R_0603, F.Cu at (51.4, 67.6)
- added R12: DNI, Resistors_SMD:R_0603_HandSoldering, F.Cu at (45.0, 101.5)
- added R13: DNI, Resistors_SMD:R_0603_HandSoldering, F.Cu at (64.0, 97.8)
- added R14: DNI, Resistors_SMD:R_0603_HandSoldering, F.Cu at (64.0, 101.8)
- added R15: DNI, Resistors_SMD:R_0603_HandSoldering, F.Cu at (45.0, 110.0)
- added R16: DNI, Resistors_SMD:R_0603_HandSoldering, F.Cu at (45.0, 114.0)
- added R17: DNI, Resistors_SMD:R_0603_HandSoldering, F.Cu at (64.0, 110.0)
- added R18: DNI, Resistors_SMD:R_0603_HandSoldering, F.Cu at (64.0, 114.0)
- added R2: 10k, Resistors_SMD:R_0603, F.Cu at (124.2, 75.3)
- added R3: DNI, Resistors_SMD:R_0603_HandSoldering, F.Cu at (45.0, 72.5)
- added R4: DNI, Resistors_SMD:R_0603_HandSoldering, F.Cu at (45.0, 76.5)
- added R5: DNI, Resistors_SMD:R_0603_HandSoldering, F.Cu at (64.2, 72.8)
- added R6: DNI, Resistors_SMD:R_0603_HandSoldering, F.Cu at (64.2, 76.8)
- added R7: DNI, Resistors_SMD:R_0603_HandSoldering, F.Cu at (45.0, 85.0)
- added R8: DNI, Resistors_SMD:R_0603_HandSoldering, F.Cu at (45.0, 89.0)
- added R9: DNI, Resistors_SMD:R_0603_HandSoldering, F.Cu at (64.2, 85.2)
- added U1001: VMEMega_no-ICSP2, arduino:VMEMegaShield_no-ICSPs, F.Cu at (25.4, 52.4)
- added U1101: TPIC2810, SMD_Packages:SO-16-N, F.Cu at (111.0, 71.8)
- added U1102: TPIC2810, SMD_Packages:SO-16-N, F.Cu at (101.2, 71.7)
- added U602: diffamp, Housings_SOIC:SOIC-14_3.9x8.7mm_Pitch1.27mm, F.Cu at (51.8, 74.5)
- added U603: diffamp, Housings_SOIC:SOIC-14_3.9x8.7mm_Pitch1.27mm, F.Cu at (71.0, 74.8)
- added U702: diffamp, Housings_SOIC:SOIC-14_3.9x8.7mm_Pitch1.27mm, F.Cu at (51.8, 87.0)
- added U703: diffamp, Housings_SOIC:SOIC-14_3.9x8.7mm_Pitch1.27mm, F.Cu at (71.0, 87.2)
- added U802: diffamp, Housings_SOIC:SOIC-14_3.9x8.7mm_Pitch1.27mm, F.Cu at (51.8, 99.5)
- added U803: diffamp, Housings_SOIC:SOIC-14_3.9x8.7mm_Pitch1.27mm, F.Cu at (71.0, 99.8)
- added U902: diffamp, Housings_SOIC:SOIC-14_3.9x8.7mm_Pitch1.27mm, F.Cu at (51.8, 112.0)
- added U903: diffamp, Housings_SOIC:SOIC-14_3.9x8.7mm_Pitch1.27mm, F.Cu at (71.0, 112.0)
- C105: value 0.33u -> 0.1u; footprint Capacitors_SMD:C_1206 -> Capacitors_SMD:C_0603
- C106: value 0.1u -> 0.33u; footprint Capacitors_SMD:C_0603 -> Capacitors_SMD:C_1206
- C301, C304, C401, C404, C501, C504: value C -> 10n
- C302, C303, C402, C403, C502, C503: value C -> 0.1u; footprint Capacitors_SMD:C_0603_HandSoldering -> Capacitors_SMD:C_0603
- C305, C306, C405, C406, C505, C506: value 0.1u -> 10n; footprint Capacitors_SMD:C_0603 -> Capacitors_SMD:C_0603_HandSoldering
- C601, C602, C603, C604, C701, C702, C703, C704, C801, C802, C803, C804, C901, C902, C903, C904: value C -> 2n
- P102: value CONN_02X30 -> CONN_02X25; footprint Pin_Headers:Pin_Header_Angled_2x30 -> Pin_Headers:Pin_Header_Angled_2x25
- P105: footprint Connect:1pin -> screw_terminals:keystone_7773
- P106: value CONN_02X18 -> CONN_01X01; footprint Pin_Headers:Pin_Header_Straight_2x18 -> screw_terminals:keystone_7773
- R301, R302, R303, R304, R401, R402, R403, R404, R501, R502, R503, R504, R601, R602, R603, R604, R701, R702, R703, R704, R801, R802, R803, R804, R901, R902, R903, R904: value 10k -> 100
- RP301, RP401: value R_PACK8 -> R_PACK4; footprint Resistors_SMD:R_Cat16-8 -> Resistors_SMD:R_Cat16-4
- moved P106 121.0 mm to (31.0, 140.8)
- moved R301 75.7 mm to (91.8, 133.6), turned to 0 degrees
- moved R302 75.0 mm to (96.8, 133.6), turned to 180 degrees
- moved C906 69.5 mm to (45.5, 112.0), turned to 0 degrees
- moved C301 67.5 mm to (87.0, 131.1)
- moved C302 66.8 mm to (94.2, 134.3), turned to 270 degrees
- moved RP301 64.5 mm to (86.8, 128.1)
- moved IC301 64.4 mm to (94.2, 128.1), turned to 90 degrees
- moved P105 64.3 mm to (31.0, 63.2)
- moved C305 62.7 mm to (87.0, 123.3), turned to 0 degrees
- moved C905 57.7 mm to (58.0, 112.0), turned to 0 degrees
- moved R304 54.8 mm to (91.8, 122.5), turned to 0 degrees
- moved R901 54.3 mm to (58.0, 114.0)
- moved C304 54.2 mm to (87.0, 133.1)
- moved R801 54.0 mm to (58.0, 101.5)
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Connections:
- net Net-(U101-Pad57) renamed +2V5
- C106 pad 1: /AV_DD -> +15V
- C107 pad 1: +15V -> /AV_DD
- C301 pad 1: Net-(C301-Pad1) -> /Aout0
- C302 pad 1: Net-(C302-Pad1) -> +15V
- C303 pad 1: Net-(C303-Pad1) -> GNDA
- C303 pad 2: GNDA -> -15V
- C304 pad 1: Net-(C304-Pad1) -> /Aout1
- C305 pad 1: +15V -> /Aout2
- C306 pad 1: GNDA -> /Aout3
- C306 pad 2: -15V -> GNDA
- C401 pad 1: Net-(C401-Pad1) -> /Aout4
- C402 pad 1: Net-(C402-Pad1) -> +15V
- C403 pad 1: Net-(C403-Pad1) -> GNDA
- C403 pad 2: GNDA -> -15V
- C404 pad 1: Net-(C404-Pad1) -> /Aout5
- C405 pad 1: +15V -> /Aout6
- C406 pad 1: GNDA -> /Aout7
- C406 pad 2: -15V -> GNDA
- C501 pad 1: Net-(C501-Pad1) -> /Aout8
- C502 pad 1: Net-(C502-Pad1) -> +15V
- C503 pad 1: Net-(C503-Pad1) -> GNDA
- C503 pad 2: GNDA -> -15V
- C504 pad 1: Net-(C504-Pad1) -> /Aout9
- C505 pad 1: +15V -> /Aout10
- C506 pad 1: GNDA -> /Aout11
- C506 pad 2: -15V -> GNDA
- IC301 pad 1: Net-(C302-Pad1) -> Net-(IC301-Pad1)
- IC301 pad 14: Net-(C303-Pad1) -> Net-(IC301-Pad13)
- IC301 pad 2: Net-(IC301-Pad2) -> Net-(IC301-Pad1)
- IC301 pad 7: Net-(C301-Pad1) -> Net-(IC301-Pad6)
- IC301 pad 8: Net-(C304-Pad1) -> Net-(IC301-Pad8)
- IC301 pad 9: Net-(IC301-Pad9) -> Net-(IC301-Pad8)
- IC401 pad 1: Net-(C402-Pad1) -> Net-(IC401-Pad1)
- IC401 pad 14: Net-(C403-Pad1) -> Net-(IC401-Pad13)
- IC401 pad 2: Net-(IC401-Pad2) -> Net-(IC401-Pad1)
- IC401 pad 7: Net-(C401-Pad1) -> Net-(IC401-Pad6)
- IC401 pad 8: Net-(C404-Pad1) -> Net-(IC401-Pad8)
- IC401 pad 9: Net-(IC401-Pad9) -> Net-(IC401-Pad8)
- IC501 pad 1: Net-(C501-Pad1) -> Net-(IC501-Pad1)
- IC501 pad 14: Net-(C504-Pad1) -> Net-(IC501-Pad13)
- IC501 pad 2: Net-(IC501-Pad2) -> Net-(IC501-Pad1)
- IC501 pad 7: Net-(C502-Pad1) -> Net-(IC501-Pad6)
- IC501 pad 8: Net-(C503-Pad1) -> Net-(IC501-Pad8)
- IC501 pad 9: Net-(IC501-Pad9) -> Net-(IC501-Pad8)
- P102 pad 10: /buffer-top/buffer_se0/OUT2 -> /Aout3
- P102 pad 11: /buffer-top/buffer_se1/OUT1 -> /Aout4
- P102 pad 12: /buffer-top/buffer_se1/OUT0 -> /Aout5
- P102 pad 13: /buffer-top/buffer_se1/OUT3 -> /Aout6
- P102 pad 14: /buffer-top/buffer_se1/OUT2 -> /Aout7
- P102 pad 15: /buffer-top/buffer_se2/OUT1 -> /Aout8
- P102 pad 16: /buffer-top/buffer_se2/OUT0 -> /Aout9
- P102 pad 17: /buffer-top/buffer_se2/OUT3 -> /Aout10
- P102 pad 18: /buffer-top/buffer_se2/OUT2 -> /Aout11
- P102 pad 19: /buffer-top/buffer3/AIN+3 -> /Ain-15
- P102 pad 20: /buffer-top/buffer3/AIN-3 -> /Ain+15
- P102 pad 21: /buffer-top/buffer3/AIN+2 -> /Ain-14
- P102 pad 22: /buffer-top/buffer3/AIN-2 -> /Ain+14
- P102 pad 23: /buffer-top/buffer3/AIN+1 -> /Ain-13
- P102 pad 24: /buffer-top/buffer3/AIN-1 -> /Ain+13
- P102 pad 25: /buffer-top/buffer3/AIN+0 -> /Ain-12
- P102 pad 26: /buffer-top/buffer3/AIN-0 -> /Ain+12
- P102 pad 27: /buffer-top/buffer2/AIN+3 -> /Ain-11
- P102 pad 28: /buffer-top/buffer2/AIN-3 -> /Ain+11
- P102 pad 29: /buffer-top/buffer2/AIN+2 -> /Ain-10
- P102 pad 3: +15V -> -15V
- P102 pad 30: /buffer-top/buffer2/AIN-2 -> /Ain+10
- P102 pad 31: /buffer-top/buffer2/AIN+1 -> /Ain-9
- P102 pad 32: /buffer-top/buffer2/AIN-1 -> /Ain+9
- P102 pad 33: /buffer-top/buffer2/AIN+0 -> /Ain-8
- P102 pad 34: /buffer-top/buffer2/AIN-0 -> /Ain+8
- P102 pad 35: /buffer-top/buffer1/AIN+3 -> /Ain-7
- P102 pad 36: /buffer-top/buffer1/AIN-3 -> /Ain+7
- P102 pad 37: /buffer-top/buffer1/AIN+2 -> /Ain-6
- P102 pad 38: /buffer-top/buffer1/AIN-2 -> /Ain+6
- P102 pad 39: /buffer-top/buffer1/AIN+1 -> /Ain-5
- P102 pad 4: -15V -> +15V
- P102 pad 40: /buffer-top/buffer1/AIN-1 -> /Ain+5
- P102 pad 41: /buffer-top/buffer1/AIN+0 -> /Ain-4
- P102 pad 42: /buffer-top/buffer1/AIN-0 -> /Ain+4
- P102 pad 43: /buffer-top/buffer0/AIN+3 -> /Ain-3
- P102 pad 44: /buffer-top/buffer0/AIN-3 -> /Ain+3
- P102 pad 45: /buffer-top/buffer0/AIN+2 -> /Ain-2
- P102 pad 46: /buffer-top/buffer0/AIN-2 -> /Ain+2
- P102 pad 47: /buffer-top/buffer0/AIN+1 -> /Ain-1
- P102 pad 48: /buffer-top/buffer0/AIN-1 -> /Ain+1
- P102 pad 49: /buffer-top/buffer0/AIN+0 -> /Ain-0
- P102 pad 50: /buffer-top/buffer0/AIN-0 -> /Ain+0
- P102 pad 7: /buffer-top/buffer_se0/OUT1 -> /Aout0
- P102 pad 8: /buffer-top/buffer_se0/OUT0 -> /Aout1
- P102 pad 9: /buffer-top/buffer_se0/OUT3 -> /Aout2
- P105 pad 1: (no net) -> Net-(P105-Pad1)
- P106 pad 1: +5V -> Net-(P106-Pad1)
- R301 pad 1: Net-(IC301-Pad5) -> /DAC_0
- R301 pad 2: GNDA -> Net-(IC301-Pad3)
- R302 pad 1: Net-(IC301-Pad3) -> /DAC_1
- R302 pad 2: GNDA -> Net-(IC301-Pad5)
- R303 pad 1: Net-(IC301-Pad12) -> /DAC_2
- R303 pad 2: GNDA -> Net-(IC301-Pad10)
- R304 pad 1: Net-(IC301-Pad10) -> /DAC_3
- R304 pad 2: GNDA -> Net-(IC301-Pad12)
- R401 pad 1: Net-(IC401-Pad5) -> /DAC_4
- R401 pad 2: GNDA -> Net-(IC401-Pad3)
- R402 pad 1: Net-(IC401-Pad3) -> /DAC_5
- R402 pad 2: GNDA -> Net-(IC401-Pad5)
- R403 pad 1: Net-(IC401-Pad12) -> /DAC_6
- R403 pad 2: GNDA -> Net-(IC401-Pad10)
- R404 pad 1: Net-(IC401-Pad10) -> /DAC_7
- R404 pad 2: GNDA -> Net-(IC401-Pad12)
- R501 pad 1: /buffer-top/buffer_se0/IN0 -> /DAC_8
- R502 pad 1: /buffer-top/buffer_se0/IN1 -> /DAC_9
- R503 pad 1: /buffer-top/buffer_se0/IN2 -> /DAC_10
- R504 pad 1: /buffer-top/buffer_se0/IN3 -> /DAC_11
- R601 pad 1: Net-(IC601-Pad5) -> Net-(C602-Pad1)
- R601 pad 2: GNDA -> /ADC_1
- R602 pad 1: Net-(IC601-Pad3) -> Net-(C603-Pad1)
- R602 pad 2: GNDA -> /ADC_2
- R603 pad 1: Net-(IC601-Pad12) -> Net-(C604-Pad1)
- R603 pad 2: GNDA -> /ADC_3
- R604 pad 1: Net-(IC601-Pad10) -> Net-(C601-Pad1)
- R604 pad 2: GNDA -> /ADC_0
- R701 pad 1: Net-(IC701-Pad5) -> Net-(C702-Pad1)
- R701 pad 2: GNDA -> /ADC_5
- R702 pad 1: Net-(IC701-Pad3) -> Net-(C703-Pad1)
- R702 pad 2: GNDA -> /ADC_6
- R703 pad 1: Net-(IC701-Pad12) -> Net-(C704-Pad1)
- R703 pad 2: GNDA -> /ADC_7
- R704 pad 1: Net-(IC701-Pad10) -> Net-(C701-Pad1)
- R704 pad 2: GNDA -> /ADC_4
- R801 pad 1: /buffer-top/buffer_se1/IN0 -> Net-(C802-Pad1)
- R801 pad 2: Net-(IC801-Pad3) -> /ADC_9
- R802 pad 1: /buffer-top/buffer_se1/IN1 -> Net-(C803-Pad1)
- R802 pad 2: Net-(IC801-Pad5) -> /ADC_10
- R803 pad 1: /buffer-top/buffer_se1/IN2 -> Net-(C804-Pad1)
- R803 pad 2: Net-(IC801-Pad10) -> /ADC_11
- R804 pad 1: /buffer-top/buffer_se1/IN3 -> Net-(C801-Pad1)
- R804 pad 2: Net-(IC801-Pad12) -> /ADC_8
- R901 pad 1: /buffer-top/buffer_se2/IN0 -> Net-(C902-Pad1)
- R901 pad 2: Net-(IC901-Pad3) -> /ADC_13
- R902 pad 1: /buffer-top/buffer_se2/IN1 -> Net-(C903-Pad1)
- R902 pad 2: Net-(IC901-Pad5) -> /ADC_14
- R903 pad 1: /buffer-top/buffer_se2/IN2 -> Net-(C904-Pad1)
- R903 pad 2: Net-(IC901-Pad10) -> /ADC_15
- R904 pad 1: /buffer-top/buffer_se2/IN3 -> Net-(C901-Pad1)
- R904 pad 2: Net-(IC901-Pad12) -> /ADC_12
- RP301 pad 1: /buffer-top/buffer0/AIN-0 -> Net-(IC301-Pad1)
- RP301 pad 2: /buffer-top/buffer0/AIN+0 -> Net-(IC301-Pad6)
- RP301 pad 3: /buffer-top/buffer0/AIN-1 -> Net-(IC301-Pad8)
- RP301 pad 4: /buffer-top/buffer0/AIN+1 -> Net-(IC301-Pad13)
- RP301 pad 5: /buffer-top/buffer0/AIN-2 -> /Aout3
- RP301 pad 6: /buffer-top/buffer0/AIN+2 -> /Aout2
- RP301 pad 7: /buffer-top/buffer0/AIN-3 -> /Aout1
- RP301 pad 8: /buffer-top/buffer0/AIN+3 -> /Aout0
- RP401 pad 1: /buffer-top/buffer1/AIN-0 -> Net-(IC401-Pad1)
- RP401 pad 2: /buffer-top/buffer1/AIN+0 -> Net-(IC401-Pad6)
- RP401 pad 3: /buffer-top/buffer1/AIN-1 -> Net-(IC401-Pad8)
- RP401 pad 4: /buffer-top/buffer1/AIN+1 -> Net-(IC401-Pad13)
- RP401 pad 5: /buffer-top/buffer1/AIN-2 -> /Aout7
- RP401 pad 6: /buffer-top/buffer1/AIN+2 -> /Aout6
- RP401 pad 7: /buffer-top/buffer1/AIN-3 -> /Aout5
- RP401 pad 8: /buffer-top/buffer1/AIN+3 -> /Aout4
- RP501 pad 1: Net-(C501-Pad1) -> Net-(IC501-Pad1)
- RP501 pad 2: Net-(C502-Pad1) -> Net-(IC501-Pad6)
- RP501 pad 3: Net-(C503-Pad1) -> Net-(IC501-Pad8)
- RP501 pad 4: Net-(C504-Pad1) -> Net-(IC501-Pad13)
- RP501 pad 5: /buffer-top/buffer_se0/OUT3 -> /Aout11
- RP501 pad 6: /buffer-top/buffer_se0/OUT2 -> /Aout10
- RP501 pad 7: /buffer-top/buffer_se0/OUT1 -> /Aout9
- RP501 pad 8: /buffer-top/buffer_se0/OUT0 -> /Aout8
- U101 pad 11: (no net) -> GNDD
- U101 pad 13: (no net) -> GNDD
- U101 pad 14: (no net) -> GNDD
- U101 pad 15: (no net) -> GNDD
- U101 pad 16: (no net) -> GNDD
- U101 pad 18: /buffer-top/buffer_se1/IN1 -> /DAC_5
- U101 pad 19: /buffer-top/buffer_se1/IN0 -> /DAC_4
- U101 pad 20: /buffer-top/buffer_se0/IN3 -> /DAC_3
- U101 pad 24: /buffer-top/buffer_se0/IN2 -> /DAC_2
- U101 pad 25: /buffer-top/buffer_se0/IN1 -> /DAC_1
- U101 pad 26: /buffer-top/buffer_se0/IN0 -> /DAC_0
- U101 pad 27: (no net) -> GNDA
- U101 pad 28: (no net) -> GNDA
- U101 pad 29: (no net) -> GNDA
- U101 pad 30: (no net) -> GNDA
- U101 pad 33: /buffer-top/buffer0/ADC0 -> /ADC_0
- U101 pad 34: /buffer-top/buffer0/ADC1 -> /ADC_1
- U101 pad 35: /buffer-top/buffer0/ADC2 -> /ADC_2
- U101 pad 36: /buffer-top/buffer0/ADC3 -> /ADC_3
- U101 pad 37: /buffer-top/buffer1/ADC0 -> /ADC_4
- U101 pad 38: /buffer-top/buffer1/ADC1 -> /ADC_5
- U101 pad 39: /buffer-top/buffer1/ADC2 -> /ADC_6
- U101 pad 40: /buffer-top/buffer1/ADC3 -> /ADC_7
- U101 pad 41: /buffer-top/buffer2/ADC0 -> /ADC_8
- U101 pad 42: /buffer-top/buffer2/ADC1 -> /ADC_9
- U101 pad 43: /buffer-top/buffer2/ADC2 -> /ADC_10
- U101 pad 44: /buffer-top/buffer2/ADC3 -> /ADC_11
- U101 pad 45: /buffer-top/buffer3/ADC0 -> /ADC_12
- U101 pad 46: /buffer-top/buffer3/ADC1 -> /ADC_13
- U101 pad 47: /buffer-top/buffer3/ADC2 -> /ADC_14
- U101 pad 48: /buffer-top/buffer3/ADC3 -> /ADC_15
- U101 pad 51: /buffer-top/buffer_se1/IN2 -> /DAC_6
- U101 pad 52: /buffer-top/buffer_se1/IN3 -> /DAC_7
- U101 pad 53: /buffer-top/buffer_se2/IN0 -> /DAC_8
- U101 pad 59: /buffer-top/buffer_se2/IN1 -> /DAC_9
- U101 pad 60: /buffer-top/buffer_se2/IN2 -> /DAC_10
- U101 pad 61: /buffer-top/buffer_se2/IN3 -> /DAC_11
- U101 pad 65: (no net) -> GNDA
Routing:
- net +15V: track 275.2 -> 546.7 mm, vias 18 -> 16
- net +5V: track 76.3 -> 317.8 mm, vias 4 -> 6
- net /buffer-top/buffer_se0/IN0: track 203.1 -> 0.00 mm, vias 2 -> 0
- net /buffer-top/buffer_se0/IN1: track 190.3 -> 0.00 mm, vias 2 -> 0
- net /buffer-top/buffer_se0/IN3: track 189.6 -> 0.00 mm
- net /buffer-top/buffer_se0/IN2: track 186.0 -> 0.00 mm, vias 2 -> 0
- net /buffer-top/buffer_se1/IN0: track 169.2 -> 0.00 mm
- net /buffer-top/buffer_se1/IN1: track 156.5 -> 0.00 mm
- net -15V: track 219.2 -> 359.2 mm, vias 8 -> 13
- net /ADC_REF: track 0.00 -> 132.6 mm, vias 0 -> 14
- net /Sheet57BE2601/Ain_os13: track 0.00 -> 114.9 mm, vias 0 -> 3
- net GNDA: track 903.7 -> 794.4 mm, vias 198 -> 140
- net /Sheet57BE2601/Ain_os12: track 0.00 -> 103.0 mm, vias 0 -> 4
- net /Sheet57BE2601/Ain_os5: track 0.00 -> 91.5 mm, vias 0 -> 4
- net /Sheet57BE2601/Ain_os4: track 0.00 -> 82.7 mm, vias 0 -> 4
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- added copper zone on In1.Cu, net GNDD
- removed copper zone on B.Cu, net +15V
- removed copper zone on F.Cu, net +5V
- removed copper zone on B.Cu, net -15V
- removed copper zone on B.Cu, net GNDD
Other:
- board size 123.2 x 100 mm -> 138.6 x 100 mm
- copper layers 2 -> 4
- board text added: "(+)"
- board text added: "0"
- board text added: "MegaDAQ v1c MFE 03/2017"
- board text removed: "+15V"
- board text removed: "-15V"
- board text removed: "AGND"
- board text removed: "MegaDAQ v1B MFE 04/2016"
