File: megaDAQ.sch (KiCad schematic (older format))
At the start: 23 parts, among them P101 CONN_02X03, P102 CONN_02X30, P103 CONN_01X01, P104 CONN_01X01, P105 CONN_01X01, P106 CONN_02X18, P107 CONN_01X10, P108 CONN_01X08, P109 CONN_01X08, P110 CONN_01X01, P111 CONN_01X01, P112 CONN_01X01, P113 CONN_01X01, P114 CONN_01X01, U101 AMC7812SPAPR, U102 LM78M05CT

Commit message: commiting version v1c, produced
Parts:
- removed P101: CONN_02X03, Pin_Headers:Pin_Header_Straight_2x03, symbol CONN_02X03
- removed P102: CONN_02X30, Pin_Headers:Pin_Header_Angled_2x30, symbol CONN_02X30
- removed P105, P110, P111, P112, P113, P114: CONN_01X01, Connect:1pin, symbol CONN_01X01
- removed P106: CONN_02X18, Pin_Headers:Pin_Header_Straight_2x18, symbol CONN_02X18
- removed P107: CONN_01X10, Pin_Headers:Pin_Header_Straight_1x10, symbol CONN_01X10
- removed P108, P109: CONN_01X08, Pin_Headers:Pin_Header_Straight_1x08, symbol CONN_01X08
- added P102: CONN_02X25, Pin_Headers:Pin_Header_Angled_2x25, symbol CONN_02X25
- added U1001: VMEMega_no-ICSP2, arduino:VMEMegaShield_no-ICSPs, symbol VMEMega_no-ICSP2
- C103: manf# (none) -> TAJY477K006RNJ
- C106: renamed from C105; manf# (none) -> 1276-1138-1-ND
- P105: renamed from P103; manf# (none) -> 7773
- P106: renamed from P104; manf# (none) -> 7773
- U101: manf# (none) -> AMC7812BSRGCR
- U102: manf# (none) -> AZ1117CH-5.0TRG1
- renumbered C107 to C105, C106 to C107
Connections:
- net labels added: !ENCJ_RST, +2V5, ADC_REF, Ain_os[0..15]
- net labels removed: 0(Rx0), 1(Tx0), 10(**), 11(**), 12(**), 13(**), 14(Tx3), 15(Rx3), 16(Tx2), 17(Rx2), 18(Tx1), 19(Rx1), 2(**), 20(SDA), 21(SCL), 22, 23, 24, 25, 26, 27, 28, 29, 3(**), 30, 31, 32, 33, 34, 35, 36, 37, 38, 39, 4(**), 40, 41, 42, 5(**), 6(**), 7(**), 8(**), 9(**), AREF, DIO0, DIO1, DIO2, DIO3, DIO4, DIO5
- wire segments 240 -> 204
- no-connect marks 56 -> 72
Other:
- note added: "Analog power for DAC outputs (+/-15V nom.)\nAV_DD is derived from here"
- note removed: "Analog power for DAC outputs (+/-12V nom.)\nAV_DD is derived from here"
- note removed: "Holes"
